File: Hardware/ogx360.brd (EAGLE design)
At the start: 97.1 x 36.5 mm, 30 parts, among them J1 USB_A_SMT_FEMALE_NS, Q1 12MHz, U1 MAX3421, U2 74HC4050, U3 MIC5219 3.3V, U4 ARDUINO_LEONARDO_MICRO, U5 ARDUINO_LEONARDO_MICRO, U6 ARDUINO_LEONARDO_MICRO, U7 ARDUINO_LEONARDO_MICRO

Commit message: HW: PCB to revision 1
Parts:
- removed F1: 6V/0.5A, SparkFun-Fuses:1206
- removed PWR: (no value), led:CHIP-LED0805
- removed Q1: 12MHz, SparkFun-Clocks:CRYSTAL-SMD-5X3.2-4PAD
- removed R5, R6, R7: 1k, rcl:R0402
- added TP1, TP2, TP3, TP4: TPTP10R, testpad:TP10R
- added Y1: 12MHz, ECS-250-18-5PX-JEM-TR:XTAL_ECS-250-18-5PX-JEM-TR
- C1, C4, C5, C7, C8: device rcl:C0402K -> rcl:C0805
- C2, C3: value 18p -> 16p; device rcl:C0402K -> rcl:C0805
- D1, D2, D3: value SOD523 -> (none); device diode:SOD523 -> diode:SOD123
- R1, R2: device rcl:R0402 -> rcl:R0805
- R3, R4: value 1k -> 2k; device rcl:R0402 -> rcl:R0805
- U1: value MAX3421 -> MAX3421ETQFP32-5MM; device SparkFun-IC-Comms:TQFP32-5MM -> my-library:TQFP32-5X5MM
- U3: value MIC5219 3.3V -> MIC5219-3.3YM5-TR; device SparkFun-IC-Power:SOT23-5 -> my-library:SOT-23-5_M5_MCH
- moved C6 6.68 mm to (18.4, 18.7), turned to 180 degrees
- moved C1 6.67 mm to (17.8, 27.9)
- moved U3 6.61 mm to (19.7, 14.0), turned to 90 degrees
- moved C7 5.46 mm to (14.6, 14.0)
- moved C8 4.46 mm to (16.8, 14.0)
- moved C2 4.41 mm to (6.67, 20.6), turned to 90 degrees
- moved C3 4.02 mm to (6.67, 24.8), turned to 270 degrees
- moved C4 3.13 mm to (12.1, 15.9), turned to 270 degrees
- moved U1 3.13 mm to (12.7, 23.5)
- moved R3 1.91 mm to (33.0, 18.4), turned to 0 degrees
- moved D1 1.71 mm to (49.5, 32.1)
- moved D2 1.62 mm to (68.6, 32.1)
- moved D3 1.59 mm to (87.0, 32.1)
- moved R2 1.14 mm to (7.62, 15.9)
- moved R1 1.00 mm to (9.84, 15.9)
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- renumbered RESET to SW1
Connections:
- net MOSI renamed AT_MOSI
- net N$1 renamed +5V_SLAVE1
- net N$3 renamed +5V_SLAVE2
- net N$4 renamed +5V_SLAVE3
- net SCK renamed AT_SCK
- net USB_RESET_IN renamed MAX_RES
- net USB_SS renamed AT_SS
- removed net MISO: U1.15, U4.P$10
- removed net MOSI_IN: U1.16, U2.2
- removed net N$13: U4.P$24, U5.P$23, U6.P$23, U7.P$23
- removed net N$138: F1.1, J1.VBUS
- removed net N$14: PWR.A, R5.1
- removed net N$2: R3.1, R6.2
- removed net N$6: R4.1, R7.2
- removed net SCK_IN: U1.13, U2.6
- removed net USB_SS_IN: U1.14, U2.4
- new net AT_RES: U2.9
- new net MAX_INT: U1.18, U4.P$15
- new net MAX_MISO: TP4.TP, U1.15, U4.P$10
- new net MAX_MOSI: TP1.TP, U1.16, U2.2
- new net MAX_SCK: TP3.TP, U1.13, U2.6
- new net MAX_SS: TP2.TP, U1.14, U2.4
- net +3V3: no longer R5.2
- net +5V: now also J1.VBUS; no longer F1.2
- net GND: no longer PWR.C
- net I2C_SCL: now also R3.1; no longer R6.1
- net I2C_SDA: now also R4.1; no longer R7.1
- net N$10: now also Y1.2; no longer Q1.3
- net N$9: now also Y1.1; no longer Q1.1
- net USB_RESET: no longer U2.9
Routing:
- net +5V: track 130.9 -> 1.59 mm, vias 6 -> 0
- net N$13: track 59.4 -> 0.00 mm
- net MAX_MISO: track 0.00 -> 37.7 mm, vias 0 -> 1
- net MISO: track 35.3 -> 0.00 mm
- net GND: track 53.9 -> 23.1 mm, vias 10 -> 17
- net MAX_SCK: track 0.00 -> 27.9 mm
- net SCK_IN: track 27.4 -> 0.00 mm
- net MAX_SS: track 0.00 -> 26.1 mm, vias 0 -> 2
- net MAX_MOSI: track 0.00 -> 26.0 mm
- net USB_SS_IN: track 25.1 -> 0.00 mm
- net MOSI_IN: track 23.1 -> 0.00 mm, vias 2 -> 0
- net MAX_INT: track 0.00 -> 22.6 mm, vias 0 -> 1
- net D_P: track 25.9 -> 11.2 mm, vias 0 -> 2
- net +3V3: track 12.3 -> 25.9 mm
- net D_N: track 25.8 -> 12.7 mm, vias 0 -> 2
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- added copper zone on layer 1, net +5V
Other:
- board text removed: "Ryzee119"
- board text removed: "ogx360"
