File: Hardware/ogx360.sch (EAGLE design)
At the start: 30 parts, among them J1 USB_A_SMT_FEMALE_NS, Q1 12MHz, U1 MAX3421, U2 74HC4050, U3 MIC5219 3.3V, U4 ARDUINO_LEONARDO_MICRO, U5 ARDUINO_LEONARDO_MICRO, U6 ARDUINO_LEONARDO_MICRO, U7 ARDUINO_LEONARDO_MICRO

Commit message: HW: PCB to revision 1
Parts:
- removed F1: 6V/0.5A, SparkFun-Fuses:PPTC_HALF-AMP
- removed PWR: (no value), led:LEDCHIP-LED0805
- removed Q1: 12MHz, SparkFun-Clocks:CRYSTALSMD-5X3.2-4PAD
- removed R5, R6, R7: 1k, rcl:R-EU_R0402
- added TP1, TP2, TP3, TP4: TPTP10R, testpad:TPTP10R
- added Y1: 12MHz, ECS-250-18-5PX-JEM-TR:ECS-250-18-5PX-JEM-TR
- C1, C4, C5, C7, C8: device rcl:C-EUC0402K -> rcl:C-EUC0805
- C2, C3: value 18p -> 16p; device rcl:C-EUC0402K -> rcl:C-EUC0805
- D1, D2, D3: value SOD523 -> (none); device diode:DIODE-SOD523 -> diode:DIODE-SOD123
- R1, R2: device rcl:R-EU_R0402 -> rcl:R-EU_R0805
- R3, R4: value 1k -> 2k; device rcl:R-EU_R0402 -> rcl:R-EU_R0805
- U1: value MAX3421 -> MAX3421ETQFP32-5MM; device SparkFun-IC-Comms:MAX3421ESMD -> my-library:MAX3421ETQFP32-5MM
- U3: value MIC5219 3.3V -> MIC5219-3.3YM5-TR; device SparkFun-IC-Power:V_REG_MIC52193.3V -> my-library:MIC5219-3.3YM5-TR
- renumbered RESET to SW1
Connections:
- net MOSI renamed AT_MOSI
- net N$1 renamed +5V_SLAVE1
- net N$3 renamed +5V_SLAVE2
- net N$4 renamed +5V_SLAVE3
- net SCK renamed AT_SCK
- net USB_RESET_IN renamed MAX_RES
- net USB_SS renamed AT_SS
- removed net MISO: U1.MISO, U4.D14/MISO
- removed net MOSI_IN: U1.MOSI, U2.1Y
- removed net N$13: U4.D0/TX, U5.D1/RX, U6.D1/RX, U7.D1/RX
- removed net N$138: F1.1, J1.VBUS
- removed net N$14: PWR.A, R5.1
- removed net N$2: R3.1, R6.2
- removed net N$6: R4.1, R7.2
- removed net SCK_IN: U1.SCK, U2.3Y
- removed net USB_SS_IN: U1.SS, U2.2Y
- new net AT_RES: U2.4A
- new net MAX_INT: U1.INT, U4.D7
- new net MAX_MISO: TP4.TP, U1.MISO, U4.D14/MISO
- new net MAX_MOSI: TP1.TP, U1.MOSI, U2.1Y
- new net MAX_SCK: TP3.TP, U1.SCK, U2.3Y
- new net MAX_SS: TP2.TP, U1.SS, U2.2Y
- net +3V3: no longer R5.2
- net +5V: now also J1.VBUS; no longer F1.2
- net GND: no longer PWR.C
- net I2C_SCL: now also R3.1; no longer R6.1
- net I2C_SDA: now also R4.1; no longer R7.1
- net N$10: now also Y1.2; no longer Q1.2
- net N$9: now also Y1.1; no longer Q1.1
- net USB_RESET: no longer U2.4A
Other:
- note added: "1"
- note added: "December 2020"
- note removed: "0"
- note removed: "500mA"
- note removed: "CONTROLLER SERIAL BUS (NOT USED)"
- note removed: "October 2018"
- moved on the sheet: C6, C7, C8, D1, D2, D3, R3, R4
